Commit message: 0726_for_ssh_changes_and_refined_rewards/RFM

File: IsaacLab_RFM/source/ext_loco/ext_loco/assets/SF_TRON1A_ARXR5ARM/assembly.urdf (robot description, URDF)
Before this commit: robot assembly, 19 links, 18 joints
Joints:
- joint gripper_fixed_joint: origin xyz=0.15 0 0 rpy=0 0 0 -> xyz=0 0 0 rpy=0 0 0

File: IsaacLab_RFM/source/ext_loco/ext_loco/assets/SF_TRON1A_ARXR5ARM/models/L5_umi.urdf (robot description, URDF)
Before this commit: robot L5_umi, 9 links, 8 joints
Joints:
- joint gripper_fixed_joint: origin xyz=0.1039414 0.0000388 0.0767217 rpy=0 0.2618 0 -> xyz=0 0 0 rpy=0 0 0

Commit message: change eef from link6 to camera

File: IsaacLab_RFM/source/ext_loco/ext_loco/assets/SF_TRON1A_ARXR5ARM/assembly.urdf (robot description, URDF)
Before this commit: robot assembly, 19 links, 18 joints
Joints:
- joint gripper_fixed_joint: origin xyz=0 0 0 rpy=0 0 0 -> xyz=0.1039414 0.0000388 0.0767217 rpy=0 0.2618 0

File: IsaacLab_RFM/source/ext_loco/ext_loco/assets/SF_TRON1A_ARXR5ARM/models/L5_umi.urdf (robot description, URDF)
Before this commit: robot L5_umi, 9 links, 8 joints
Joints:
- joint gripper_fixed_joint: origin xyz=0 0 0 rpy=0 0 0 -> xyz=0.1039414 0.0000388 0.0767217 rpy=0 0.2618 0

File: tron1_ws/src/tron1-rl-deploy-arm/src/robot-description/pointfoot/SF_TRON1A_ARX5ARM/urdf/assembly.urdf (robot description, URDF)
Before this commit: robot assembly, 26 links, 25 joints
Links:
- added link eef_link
Joints:
- added joint eef_camera_fixed_joint: type fixed, parent link6, child eef_link, origin xyz=0.1039414 0.0000388 0.0767217 rpy=0 0.2618 0
